Commit message: fixed urdfs to work with amiga

File: pybullet_tree_sim/urdf/robot/generic/robot_old.urdf.xacro (robot description, xacro)
@@ -123,17 +123,9 @@
                 />
             </xacro:if>
-            <xacro:if value="${ str(resolved_part) == 'amiga' }">
-                <xacro:include filename="$(arg urdf_base_path)/base_mounts/farm-ng/macro/amiga_macro.urdf.xacro"/>
-                <xacro:amiga_macro
-                    amiga_prefix="amiga__"
-                    amiga_parent="${resolved_parent_part}"
-                    mesh_base_path="$(arg mesh_base_path)"
-                />
-            </xacro:if>
-            <!-- Mock Pruner -->
             <xacro:if value="${ str(resolved_part) == 'mock_pruner' }">
                 <xacro:include filename="$(arg urdf_base_path)/end_effectors/mock_pruner/macro/mock_pruner_macro.urdf.xacro"/>
                 <!-- Args -->
                 <xacro:arg name="mock_pruner_prefix" default="mock_pruner__" />
+                <xacro:arg name="mesh_base_path" default="" />
                 <xacro:arg name="tof0_offset" default="0.1 0.0 0.142" />
                 <xacro:arg name="tof1_offset" default="-0.1 0.0 0.142"/>

File: pybullet_tree_sim/urdf/tmp/robot.urdf (robot description, URDF)
Before this commit: robot pruning_robot, 27 links, 26 joints
Links:
- added link amiga__base
- added link amiga__body, mass 40.0; collision box size=0.25 0.25 0.25; collision box size=1.132 0.6 0.2
- added link amiga__tool0
Joints:
- added joint amiga__base--amiga__body: type fixed, parent amiga__base, child amiga__body, origin xyz=0 0 0 rpy=0 0 0
- added joint amiga__body--amiga__tool0: type fixed, parent amiga__body, child amiga__tool0, origin xyz=-0.225 0.323256 1.09810607 rpy=0.0 0.0 -3.9269908169872414
- added joint world--amiga__base: type fixed, parent world, child amiga__base, origin xyz=0 0 0 rpy=0 0 0
