Commit message: beginning of major URDF refactor

File: pybullet_tree_sim/urdf/end_effectors/mock_pruner/macro/mock_pruner_macro.urdf.xacro (robot description, xacro)
@@ -46,15 +46,15 @@
         <!--     Joints        -->
         <!-- ================== -->
-        <joint name="${eef_parent}tool0--${eef_prefix}base_joint" type="fixed">
+        <joint name="${eef_parent}tool0--${eef_prefix}base" type="fixed">
             <origin xyz="0 0 0" rpy="0 0 0"/>
             <parent link="${eef_parent}tool0"/>
             <child link="${eef_prefix}base"/>
         </joint>
-        <joint name="${eef_prefix}base--camera0_joint" type="fixed">
+        <joint name="${eef_prefix}base--camera0" type="fixed">
             <origin xyz="0 0 0" rpy="0 0 0"/>
             <parent link="${eef_prefix}base" />
             <child link="${eef_prefix}camera0" />
         </joint>
-        <joint name="${eef_prefix}base--tof0_joint" type="fixed">
+        <joint name="${eef_prefix}base--tof0" type="fixed">
             <!-- <xacro:insert_block name="origin"/> -->
             <origin xyz="${tof0_offset} 0 0" rpy="0 0 0"/>
@@ -62,10 +62,10 @@
             <child link="${eef_prefix}tof0" />
         </joint>
-        <joint name="${eef_prefix}base--tof1_joint" type="fixed">
+        <joint name="${eef_prefix}base--tof1" type="fixed">
             <origin xyz="${tof1_offset} 0 0" rpy="0 0 0"/>
             <parent link="${eef_prefix}base" />
             <child link="${eef_prefix}tof1" />
         </joint>
-        <joint name="${eef_prefix}base--${eef_prefix}tool0" type="fixed">
+        <joint name="${eef_prefix}base--tool0" type="fixed">
             <origin xyz="0 0 0" rpy="0 0 0"/>
             <parent link="${eef_prefix}base" />

File: pybullet_tree_sim/urdf/robot/generic/robot.urdf.xacro (robot description, xacro)
@@ -3,188 +3,131 @@
     <!-- robot name parameter -->
     <xacro:arg name="name" default="pruning_robot"/>
-    <!-- <xacro:arg name="robot_parent" default="world" /> -->
-    <xacro:property name="base_attachment_parent" value="world"/>
-    <xacro:property name="robot_arm_parent" value="world"/>
-    <xacro:property name="end_effector_parent" value="world"/>
-    <!-- create link fixed to the "world" -->
-    <link name="world" />
-    <!-- Base attachment -->
-    <xacro:arg name="base_type" default="" />
-    <xacro:if value="${ '$(arg base_type)' == 'linear_slider' }" >
-        <!-- linear slider -->
-        <xacro:include filename="$(find linear_slider_description)/urdf/macro/linear_slider_base.urdf.xacro" />
-        <xacro:arg name="linear_slider_parent" default="${base_attachment_parent}"/>
-        <xacro:arg name="linear_slider_robot_ip" default="169.254.57.177"/> <!-- TODO: add this into the macro, but instead get from yaml file-->
-        <xacro:arg name="base_prefix" default="linear_slider__" />
-        <xacro:arg name="use_mock_hardware" default="false" />
-        <xacro:arg name="mock_sensor_commands" default="false" />
-        <xacro:arg name="sim_gazebo" default="false" />
-        <xacro:arg name="sim_gazebo_classic" default="false"/>
-        <!-- Set slider moving base as arm parent joint -->
-        <xacro:property name="robot_arm_parent" value="$(arg base_prefix)tool0" />
-        <xacro:linear_slider
-            parent="$(arg linear_slider_parent)"
-            prefix="$(arg base_prefix)"
-            sim_gazebo="$(arg sim_gazebo)"
-            sim_gazebo_classic="$(arg sim_gazebo_classic)"
-            use_mock_hardware="$(arg use_mock_hardware)"
-            mock_sensor_commands="$(arg mock_sensor_commands)"
-        />
-    </xacro:if>
-    <xacro:if value="${ '$(arg base_type)' == 'farm-ng' }" >
-        <!-- <xacro:include filename="$(find farm-ng)/urdf" /> -->
-    </xacro:if>
-    <!-- Robot arm type. Current types are UR and Franka Emika -->
-    <xacro:arg name="arm_type" default="arm_type" />
-    <xacro:if value="${ '$(arg arm_type)' == 'ur5e' }">
-        <xacro:include filename="$(find ur_description)/urdf/ur_macro.xacro"/>
-        <!-- UR -->
-        <!-- possible 'ur_type' values: ur3, ur3e, ur5, ur5e, ur10, ur10e, ur16e, ur20, ur30 -->
-        <!-- the default value should raise an error in case this was called without defining the type -->
-        <xacro:arg name="ur_type" default="$(arg arm_type)"/>
-        <xacro:arg name="ur_parent" default="${robot_arm_parent}"/>
-        <!-- parameters -->
-        <xacro:arg name="tf_prefix" default="$(arg arm_type)__" />
-        <xacro:arg name="joint_limit_params" default="$(find ur_description)/config/$(arg ur_type)/joint_limits.yaml"/>
-        <xacro:arg name="kinematics_params" default="$(find ur_description)/config/$(arg ur_type)/default_kinematics.yaml"/>
-        <xacro:arg name="physical_params" default="$(find ur_description)/config/$(arg ur_type)/physical_parameters.yaml"/>
-        <xacro:arg name="visual_params" default="$(find ur_description)/config/$(arg ur_type)/visual_parameters.yaml"/>
-        <xacro:arg name="transmission_hw_interface" default=""/>
-        <xacro:arg name="safety_limits" default="false"/>
-        <xacro:arg name="safety_pos_margin" default="0.15"/>
-        <xacro:arg name="safety_k_position" default="20"/>
-        <!-- ros2_control related parameters -->
-        <xacro:arg name="headless_mode" default="false" />
-        <xacro:arg name="robot_ip" default="0.0.0.0" />
-        <xacro:arg name="script_filename" default=""/>
-        <xacro:arg name="output_recipe_filename" default=""/>
-        <xacro:arg name="input_recipe_filename" default=""/>
-        <xacro:arg name="reverse_ip" default="0.0.0.0"/>
-        <xacro:arg name="script_command_port" default="50004"/>
-        <xacro:arg name="reverse_port" default="50001"/>
-        <xacro:arg name="script_sender_port" default="50002"/>
-        <xacro:arg name="trajectory_port" default="50003"/>
-        <!--   tool communication related parameters-->
-        <xacro:arg name="use_tool_communication" default="false" />
-        <xacro:arg name="tool_voltage" default="0" />
-        <xacro:arg name="tool_parity" default="0" />
-        <xacro:arg name="tool_baud_rate" default="115200" />
-        <xacro:arg name="tool_stop_bits" default="1" />
-        <xacro:arg name="tool_rx_idle_chars" default="1.5" />
-        <xacro:arg name="tool_tx_idle_chars" default="3.5" />
-        <xacro:arg name="tool_device_name" default="/tmp/ttyUR" />
-        <xacro:arg name="tool_tcp_port" default="54321" />
-            <!-- Simulation parameters -->
-        <xacro:arg name="use_fake_hardware" default="false" />
-        <xacro:arg name="fake_sensor_commands" default="false" />
-        <xacro:arg name="sim_gazebo" default="false" />
-        <xacro:arg name="sim_ignition" default="false" />
-        <xacro:arg name="simulation_controllers" default="" />
-        <!-- initial position for simulations (Fake Hardware, Gazebo, Ignition) -->
-        <xacro:arg name="initial_positions_file" default="$(find ur_description)/config/initial_positions.yaml"/>
-        <!-- convert to property to use substitution in function -->
-        <xacro:property name="initial_positions_file" default="$(arg initial_positions_file)"/>
-        <!-- arm -->
-        <xacro:ur_robot
-            name="$(arg name)"
-            tf_prefix="$(arg tf_prefix)"
-            parent="$(arg ur_parent)"
-            joint_limits_parameters_file="$(arg joint_limit_params)"
-            kinematics_parameters_file="$(arg kinematics_params)"
-            physical_parameters_file="$(arg physical_params)"
-            visual_parameters_file="$(arg visual_params)"
-            transmission_hw_interface="$(arg transmission_hw_interface)"
-            safety_limits="$(arg safety_limits)"
-            safety_pos_margin="$(arg safety_pos_margin)"
-            safety_k_position="$(arg safety_k_position)"
-            use_fake_hardware="$(arg use_fake_hardware)"
-            fake_sensor_commands="$(arg fake_sensor_commands)"
-            sim_gazebo="$(arg sim_gazebo)"
-            sim_ignition="$(arg sim_ignition)"
-            headless_mode="$(arg headless_mode)"
-            initial_positions="${xacro.load_yaml(initial_positions_file)}"
-            use_tool_communication="$(arg use_tool_communication)"
-            tool_voltage="$(arg tool_voltage)"
-            tool_parity="$(arg tool_parity)"
-            tool_baud_rate="$(arg tool_baud_rate)"
-            tool_stop_bits="$(arg tool_stop_bits)"
-            tool_rx_idle_chars="$(arg tool_rx_idle_chars)"
-            tool_tx_idle_chars="$(arg tool_tx_idle_chars)"
-            tool_device_name="$(arg tool_device_name)"
-            tool_tcp_port="$(arg tool_tcp_port)"
-            robot_ip="$(arg robot_ip)"
-            script_filename="$(arg script_filename)"
-            output_recipe_filename="$(arg output_recipe_filename)"
-            input_recipe_filename="$(arg input_recipe_filename)"
-            reverse_ip="$(arg reverse_ip)"
-            script_command_port="$(arg script_command_port)"
-            reverse_port="$(arg reverse_port)"
-            script_sender_port="$(arg script_sender_port)"
-            trajectory_port="$(arg trajectory_port)"
-            >
-            <origin xyz="0 0 0" rpy="0 0 0" />          <!-- position robot in the world -->
-        </xacro:ur_robot>
-        <!-- Update end-effector parent -->
-        <xacro:property name="end_effector_parent" value="$(arg tf_prefix)tool0"/>
-    </xacro:if>
-    <xacro:if value="${ '$(arg arm_type)' == 'fr3' }">
-        <xacro:include filename="$(find franka_description)/robots/common/franka_robot.xacro"/>
-        <!-- Name for this robot -->
-        <xacro:arg name="arm_id" default="fr3" />
-        <!-- Should an end-effector be mounted at the flange?" -->
-        <xacro:arg name="hand" default="true" />
-        <!-- Which end-effector would be mounted at the flange?" -->
-        <xacro:arg name="ee_id" default="franka_hand" />
-        <!-- Should self-collision be enabled? -->
-        <xacro:arg name="with_sc" default="false" />
-        <!-- Is the robot being controlled with ros2_control?" -->
-        <xacro:arg name="ros2_control" default="false" />
-        <!-- IP address or hostname of the robot" -->
-        <xacro:arg name="robot_ip" default="" />
-        <!-- Should a fake hardware be used? -->
-        <xacro:arg name="use_fake_hardware" default="false" />
-        <!-- Should fake sensors be used? -->
-        <xacro:arg name="fake_sensor_commands" default="false" />
-        <!-- Should the robot be spawned in Gazebo?" -->
-        <xacro:arg name="gazebo" default="false" />
-        <!-- Should the robot be spawned in Gazebo with effort interfaces?" -->
-        <xacro:arg name="gazebo_effort" default="false" />
-        <xacro:franka_robot arm_id="$(arg arm_id)"
-                            joint_limits="${xacro.load_yaml('$(find franka_description)/robots/$(arg arm_id)/joint_limits.yaml')}"
-                            inertials="${xacro.load_yaml('$(find franka_description)/robots/$(arg arm_id)/inertials.yaml')}"
-                            kinematics="${xacro.load_yaml('$(find franka_description)/robots/$(arg arm_id)/kinematics.yaml')}"
-                            dynamics="${xacro.load_yaml('$(find franka_description)/robots/$(arg arm_id)/dynamics.yaml')}"
-                            gazebo="$(arg gazebo)"
-                            hand="$(arg hand)"
-                            ee_id="$(arg ee_id)"
-                            with_sc="$(arg with_sc)"
-                            ros2_control="$(arg ros2_control)"
-                            robot_ip="$(arg robot_ip)"
-                            use_fake_hardware="$(arg use_fake_hardware)"
-                            fake_sensor_commands="$(arg fake_sensor_commands)"
-                            gazebo_effort="$(arg gazebo_effort)">
-        </xacro:franka_robot>
-        <!-- <xacro:property name="end_effector_parent" value="$(arg fr3_prefix)tool0"/> -->
-    </xacro:if>
-    <!-- Robot arm base/eef attachments -->
-    <xacro:arg name="end_effector_type" default=""/> -->
-    <xacro:if value="${ '$(arg eef_type)' == 'apple_picker' }">
-    </xacro:if>
-    <xacro:if value="${ '$(arg eef_type)' == 'mock_pruner' }" >
-        <xacro:include filename="../../end_effectors/mock_pruner/macro/mock_pruner_macro.urdf.xacro"/>
-        <!-- Args -->
-        <xacro:arg name="eef_parent" default="${end_effector_parent}" />
-        <xacro:arg name="eef_prefix" default="mock_pruner__" />
-        <xacro:arg name="tof0_offset_x" default='0.02'/>
-        <xacro:arg name="tof1_offset_x" default='-0.02'/>
-        <xacro:arg name="mesh_base_path" default="/home/luke/dev/pybullet/pybullet-tree-sim/pybullet_tree_sim/meshes"/>
-        <xacro:mock_pruner_macro
-            eef_prefix="$(arg eef_prefix)"
-            eef_parent="$(arg eef_parent)"
-            tof0_offset='$(arg tof0_offset_x)'
-            tof1_offset='$(arg tof1_offset_x)'
-            camera_offset=''
-            mesh_base_path='$(arg mesh_base_path)'
-        />
-    </xacro:if>
+    <xacro:arg name="robot_stack_qty" default='0'/>
+    <!-- generate generic robot with stack_qty number of links, link parents -->
+    <xacro:macro name='arg_assignment_loop' params='stack_qty'>
+        <xacro:if value="${stack_qty}">
+            <xacro:arg name="parent${stack_qty - 1}" default="world"/>
+            <xacro:arg name="robot_part${stack_qty - 1}" default="world"/>
+            <xacro:arg_assignment_loop stack_qty="${stack_qty - 1}"/>
+        </xacro:if>
+    </xacro:macro>
+    <xacro:arg_assignment_loop stack_qty="$(arg robot_stack_qty)"/>
+    <xacro:macro name="main_loop" params="stack_qty">
+        <xacro:if value="${stack_qty}">
+            <!-- Generic robot properties -->
+            <xacro:property name='resolved_robot_part' value="$(arg robot_part${stack_qty - 1})"/>
+            <xacro:property name='resolved_parent_part' value="$(arg parent${stack_qty - 1})"/>
+            <xacro:property name='resolved_parent_link' value="${resolved_parent_part}__tool0"/>
+            <xacro:if value="${stack_qty == 1}">
+                <!-- connect to world -->
+                <link name="world"/>
+                <!-- <xacro:property name="parent${stack_qty - 1}" value='world'/> -->
+                <joint name="world--link${stack_qty - 2}">
+                    <parent value="world"/>
+                    <child value="link${stack_qty - 1}"/>
+                    <origin xyz="0.0 0.0 0.0" rpy="0.0 0.0 0.0"/>
+                </joint>
+            </xacro:if>
+            <xacro:unless value="${stack_qty == 1}">
+                <!-- <link name='${str(resolved_robot_part)}'/> -->
+                <!-- UR5e -->
+                <xacro:if value="${ str(resolved_robot_part) == 'ur5e' }">
+                    <xacro:include filename="$(find ur_description)/urdf/ur_macro.xacro"/>
+                    <xacro:arg name="ur_type" default='ur5e'/>
+                    <xacro:arg name="ur_prefix" default='$(arg ur_type)__'/>
+                    <xacro:arg name="joint_limit_params" default="$(find ur_description)/config/$(arg ur_type)/joint_limits.yaml"/>
+                    <xacro:arg name="kinematics_params" default="$(find ur_description)/config/$(arg ur_type)/default_kinematics.yaml"/>
+                    <xacro:arg name="physical_params" default="$(find ur_description)/config/$(arg ur_type)/physical_parameters.yaml"/>
+                    <xacro:arg name="visual_params" default="$(find ur_description)/config/$(arg ur_type)/visual_parameters.yaml"/>
+                    <xacro:arg name="transmission_hw_interface" default=""/>
+                    <xacro:arg name="safety_limits" default="false"/>
+                    <xacro:arg name="safety_pos_margin" default="0.15"/>
+                    <xacro:arg name="safety_k_position" default="20"/>
+                    <!-- ros2_control related parameters -->
+                    <xacro:arg name="headless_mode" default="false" />
+                    <xacro:arg name="robot_ip" default="0.0.0.0" />
+                    <xacro:arg name="script_filename" default=""/>
+                    <xacro:arg name="output_recipe_filename" default=""/>
+                    <xacro:arg name="input_recipe_filename" default=""/>
+                    <xacro:arg name="reverse_ip" default="0.0.0.0"/>
+                    <xacro:arg name="script_command_port" default="50004"/>
+                    <xacro:arg name="reverse_port" default="50001"/>
+                    <xacro:arg name="script_sender_port" default="50002"/>
+                    <xacro:arg name="trajectory_port" default="50003"/>
+                    <!--   tool communication related parameters-->
+                    <xacro:arg name="use_tool_communication" default="false" />
+                    <xacro:arg name="tool_voltage" default="0" />
+                    <xacro:arg name="tool_parity" default="0" />
+                    <xacro:arg name="tool_baud_rate" default="115200" />
+                    <xacro:arg name="tool_stop_bits" default="1" />
+                    <xacro:arg name="tool_rx_idle_chars" default="1.5" />
+                    <xacro:arg name="tool_tx_idle_chars" default="3.5" />
+                    <xacro:arg name="tool_device_name" default="/tmp/ttyUR" />
+                    <xacro:arg name="tool_tcp_port" default="54321" />
+                        <!-- Simulation parameters -->
+                    <xacro:arg name="use_fake_hardware" default="false" />
+                    <xacro:arg name="fake_sensor_commands" default="false" />
+                    <xacro:arg name="sim_gazebo" default="false" />
+                    <xacro:arg name="sim_ignition" default="false" />
+                    <xacro:arg name="simulation_controllers" default="" />
+                    <!-- initial position for simulations (Fake Hardware, Gazebo, Ignition) -->
+                    <xacro:arg name="initial_positions_file" default="$(find ur_description)/config/initial_positions.yaml"/>
+                    <!-- convert to property to use substitution in function -->
+                    <xacro:property name="initial_positions_file" default="$(arg initial_positions_file)"/>
+                    <!-- arm -->
+                    <xacro:ur_robot
+                        name="$(arg name)"
+                        tf_prefix="$(arg ur_prefix)"
+                        parent="${resolved_parent_part}"
+                        joint_limits_parameters_file="$(arg joint_limit_params)"
+                        kinematics_parameters_file="$(arg kinematics_params)"
+                        physical_parameters_file="$(arg physical_params)"
+                        visual_parameters_file="$(arg visual_params)"
+                        transmission_hw_interface="$(arg transmission_hw_interface)"
+                        safety_limits="$(arg safety_limits)"
+                        safety_pos_margin="$(arg safety_pos_margin)"
+                        safety_k_position="$(arg safety_k_position)"
+                        use_fake_hardware="$(arg use_fake_hardware)"
+                        fake_sensor_commands="$(arg fake_sensor_commands)"
+                        sim_gazebo="$(arg sim_gazebo)"
+                        sim_ignition="$(arg sim_ignition)"
+                        headless_mode="$(arg headless_mode)"
+                        initial_positions="${xacro.load_yaml(initial_positions_file)}"
+                        use_tool_communication="$(arg use_tool_communication)"
+                        tool_voltage="$(arg tool_voltage)"
+                        tool_parity="$(arg tool_parity)"
+                        tool_baud_rate="$(arg tool_baud_rate)"
+                        tool_stop_bits="$(arg tool_stop_bits)"
+                        tool_rx_idle_chars="$(arg tool_rx_idle_chars)"
+                        tool_tx_idle_chars="$(arg tool_tx_idle_chars)"
+                        tool_device_name="$(arg tool_device_name)"
+                        tool_tcp_port="$(arg tool_tcp_port)"
+                        robot_ip="$(arg robot_ip)"
+                        script_filename="$(arg script_filename)"
+                        output_recipe_filename="$(arg output_recipe_filename)"
+                        input_recipe_filename="$(arg input_recipe_filename)"
+                        reverse_ip="$(arg reverse_ip)"
+                        script_command_port="$(arg script_command_port)"
+                        reverse_port="$(arg reverse_port)"
+                        script_sender_port="$(arg script_sender_port)"
+                        trajectory_port="$(arg trajectory_port)"
+                        >
+                        <origin xyz="0 0 0" rpy="0 0 0" />          <!-- position robot in the world -->
+                    </xacro:ur_robot>
+                </xacro:if>
+                <!-- Robot cart -->
+                <xacro:if value="${ str(resolved_robot_part) == 'cart' }">
+                    <xacro:include filename="../../base_mounts/cart/cart_macro.urdf.xacro"/>
+                    <xacro:cart_macro
+                        cart_prefix="cart__"
+                        cart_parent="$(arg parent${stack_qty - 1})"
+                    />
+                </xacro:if>
+                <!-- <link name="$(arg robot_part${stack_qty - 1})" /> -->
+            </xacro:unless>
+            <!-- call macro recursively -->
+            <xacro:main_loop stack_qty="${stack_qty - 1}"/>
+        </xacro:if>
+    </xacro:macro>
+    <xacro:main_loop stack_qty="$(arg robot_stack_qty)"/>
 </robot>
