Commit message: beginning of major URDF refactor

File: pybullet_tree_sim/urdf/robot/generic/test.urdf (robot description, URDF)
Before this commit: robot pruning_robot, 23 links, 22 joints
Links:
- removed link linear_slider__base
- removed link linear_slider__base_link
- removed link linear_slider__flange
- removed link linear_slider__moving_base
- removed link linear_slider__tool0
- removed link mock_pruner__base
- removed link mock_pruner__camera0
- removed link mock_pruner__tof0
- removed link mock_pruner__tof1
- removed link mock_pruner__tool0
- removed link ur5e__base
- removed link ur5e__base_link
- removed link ur5e__base_link_inertia
- removed link ur5e__flange
- removed link ur5e__forearm_link
- removed link ur5e__ft_frame
- removed link ur5e__shoulder_link
- removed link ur5e__tool0
- removed link ur5e__upper_arm_link
- removed link ur5e__wrist_1_link
- removed link ur5e__wrist_2_link
- removed link ur5e__wrist_3_link
- added link link1
- added link link2
Joints:
- removed joint linear_slider__base_joint
- removed joint linear_slider__base_link__base_joint
- removed joint linear_slider__flange__tool0_joint
- removed joint linear_slider__joint1
- removed joint linear_slider__moving_base__flange_joint
- removed joint mock_pruner__base--camera0_joint
- removed joint mock_pruner__base--mock_pruner__tool0
- removed joint mock_pruner__base--tof0_joint
- removed joint mock_pruner__base--tof1_joint
- removed joint ur5e__base_joint
- removed joint ur5e__base_link-base_fixed_joint
- removed joint ur5e__base_link-base_link_inertia
- removed joint ur5e__elbow_joint
- removed joint ur5e__flange-tool0
- removed joint ur5e__shoulder_lift_joint
- removed joint ur5e__shoulder_pan_joint
- removed joint ur5e__tool0--mock_pruner__base_joint
- removed joint ur5e__wrist_1_joint
- removed joint ur5e__wrist_2_joint
- removed joint ur5e__wrist_3-flange
- removed joint ur5e__wrist_3_joint
- removed joint ur5e__wrist_3_link-ft_frame
- added joint link1--link0: type None, parent , child , origin xyz=0.0 0.0 0.0 rpy=0.0 0.0 0.0
- added joint link2--link1: type None, parent , child , origin xyz=0.0 0.0 0.0 rpy=0.0 0.0 0.0
- added joint world--link-1: type None, parent , child , origin xyz=0.0 0.0 0.0 rpy=0.0 0.0 0.0

File: pybullet_tree_sim/urdf/tmp/robot.urdf (robot description, URDF)
Before this commit: robot pruning_robot, 18 links, 17 joints
Links:
- removed link mock_pruner__base
- removed link mock_pruner__camera0
- removed link mock_pruner__tof0
- removed link mock_pruner__tof1
- removed link mock_pruner__tool0
- removed link ur5e__base
- removed link ur5e__base_link
- removed link ur5e__base_link_inertia
- removed link ur5e__flange
- removed link ur5e__forearm_link
- removed link ur5e__ft_frame
- removed link ur5e__shoulder_link
- removed link ur5e__tool0
- removed link ur5e__upper_arm_link
- removed link ur5e__wrist_1_link
- removed link ur5e__wrist_2_link
- removed link ur5e__wrist_3_link
- added link mock_pruner
- added link ur5e
Joints:
- removed joint mock_pruner__base--camera0_joint
- removed joint mock_pruner__base--mock_pruner__tool0
- removed joint mock_pruner__base--tof0_joint
- removed joint mock_pruner__base--tof1_joint
- removed joint ur5e__base_joint
- removed joint ur5e__base_link-base_fixed_joint
- removed joint ur5e__base_link-base_link_inertia
- removed joint ur5e__elbow_joint
- removed joint ur5e__flange-tool0
- removed joint ur5e__shoulder_lift_joint
- removed joint ur5e__shoulder_pan_joint
- removed joint ur5e__tool0--mock_pruner__base_joint
- removed joint ur5e__wrist_1_joint
- removed joint ur5e__wrist_2_joint
- removed joint ur5e__wrist_3-flange
- removed joint ur5e__wrist_3_joint
- removed joint ur5e__wrist_3_link-ft_frame
- added joint mock_pruner--ur5e: type None, parent , child , origin xyz=0.0 0.0 0.0 rpy=0.0 0.0 0.0
- added joint ur5e--cart: type None, parent , child , origin xyz=0.0 0.0 0.0 rpy=0.0 0.0 0.0
- added joint world--link-1: type None, parent , child , origin xyz=0.0 0.0 0.0 rpy=0.0 0.0 0.0

Commit message: added dynamic building of the urdf. needs testing

File: pybullet_tree_sim/urdf/end_effectors/mock_pruner/macro/mock_pruner_macro.urdf.xacro (robot description, xacro)
@@ -6,5 +6,5 @@
     <!-- <xacro:property name="end_effector_parent" value="" /> -->
     <!-- Materials -->
-    <xacro:macro name="mock_pruner_macro" params="eef_prefix eef_parent tof0_offset tof1_offset camera_offset mesh_base_path">
+    <xacro:macro name="mock_pruner_macro" params="parent_link eef_prefix tof0_offset tof1_offset camera_offset mesh_base_path">
         <!-- ================== -->
         <!--     Properties     -->
@@ -46,7 +46,7 @@
         <!--     Joints        -->
         <!-- ================== -->
-        <joint name="${eef_parent}tool0--${eef_prefix}base" type="fixed">
+        <joint name="${parent_link}--${eef_prefix}base" type="fixed">
             <origin xyz="0 0 0" rpy="0 0 0"/>
-            <parent link="${eef_parent}tool0"/>
+            <parent link="${parent_link}"/>
             <child link="${eef_prefix}base"/>
         </joint>

File: pybullet_tree_sim/urdf/end_effectors/mock_pruner/mock_pruner.urdf.xacro (robot description, xacro)
@@ -4,27 +4,23 @@
     <link name="world" />
     <!-- Args -->
-    <xacro:arg name="eef_parent" default="world" />
-    <xacro:arg name="eef_prefix" default="mock_pruner__" />
+    <xacro:arg name="mock_pruner_parent_link" default="world" />
+    <xacro:arg name="mock_pruner_prefix" default="mock_pruner__" />
+    <xacro:arg name="mesh_base_path" default="" />
     <xacro:arg name="tof0_offset_x" default="0.02" />
     <xacro:arg name="tof1_offset_x" default="-0.02" />
     <!-- mock_pruner macro -->
     <xacro:include filename="./macro/mock_pruner_macro.urdf.xacro" />
-    <!-- <xacro:arg name="parent" default="world" />
-    <xacro:arg name="prefix" default="''" />
-    <xacro:arg name="use_mock_hardware" default="false" />
-    <xacro:arg name="mock_sensor_commands" default="false" />
-    <xacro:arg name="sim_gazebo" default="false" />
-    <xacro:arg name="sim_gazebo_classic" default="false"/> -->
     <xacro:mock_pruner_macro
-        eef_prefix="$(arg eef_prefix)"
-        eef_parent="$(arg eef_parent)"
+        parent_link="$(arg mock_pruner_parent_link)"
+        eef_prefix="$(arg mock_pruner_prefix)"
         tof0_offset='$(arg tof0_offset_x)'
         tof1_offset='$(arg tof1_offset_x)'
+        mesh_base_path="$(arg mesh_base_path)"
         camera_offset=''
     />
-    <joint name="world__$(arg eef_prefix)base" type="fixed">
+    <joint name="world--$(arg mock_pruner_prefix)base" type="fixed">
         <origin xyz="0.0 180.0 0.0" rpy="0 0 0"/>
         <parent link="world" />
-        <child link="$(arg eef_prefix)base" />
+        <child link="$(arg mock_pruner_prefix)base" />
     </joint>
 </robot>

File: pybullet_tree_sim/urdf/robot/generic/robot.urdf.xacro (robot description, xacro)
@@ -1,7 +1,11 @@
 <?xml version ="1.0"?>
 <robot xmlns:xacro="http://wiki.ros.org/xacro" name="pruning_robot">
+    <!-- WORLD LINK -->
+    <link name="world"/>
     <!-- robot name parameter -->
     <xacro:arg name="name" default="pruning_robot"/>
     <xacro:arg name="robot_stack_qty" default='0'/>
+    <xacro:arg name="mesh_base_path" default=''/>
+    <xacro:arg name="urdf_base_path" default=''/>
     <!-- generate generic robot with stack_qty number of links, link parents -->
     <xacro:macro name='arg_assignment_loop' params='stack_qty'>
@@ -16,114 +20,125 @@
         <xacro:if value="${stack_qty}">
             <!-- Generic robot properties -->
-            <xacro:property name='resolved_robot_part' value="$(arg robot_part${stack_qty - 1})"/>
+            <xacro:property name='resolved_part' value="$(arg robot_part${stack_qty - 1})"/>
+            <xacro:property name='resolved_part_base' value="${resolved_part}__base}"/>
             <xacro:property name='resolved_parent_part' value="$(arg parent${stack_qty - 1})"/>
             <xacro:property name='resolved_parent_link' value="${resolved_parent_part}__tool0"/>
-            <xacro:if value="${stack_qty == 1}">
-                <!-- connect to world -->
-                <link name="world"/>
-                <!-- <xacro:property name="parent${stack_qty - 1}" value='world'/> -->
-                <joint name="world--link${stack_qty - 2}">
-                    <parent value="world"/>
-                    <child value="link${stack_qty - 1}"/>
-                    <origin xyz="0.0 0.0 0.0" rpy="0.0 0.0 0.0"/>
-                </joint>
+            <!-- <xacro:unless value="${stack_qty == 1}"> -->
+            <!-- <link name="${resolved_part}"/> -->
+            <!-- <link name='${str(resolved_robot_part)}'/> -->
+            <!-- UR5e -->
+            <xacro:if value="${ str(resolved_part) == 'ur5e' }">
+                <xacro:include filename="$(find ur_description)/urdf/ur_macro.xacro"/>
+                <xacro:arg name="ur_type" default='ur5e'/>
+                <xacro:arg name="ur_prefix" default='$(arg ur_type)__'/>
+                <xacro:arg name="joint_limit_params" default="$(find ur_description)/config/$(arg ur_type)/joint_limits.yaml"/>
+                <xacro:arg name="kinematics_params" default="$(find ur_description)/config/$(arg ur_type)/default_kinematics.yaml"/>
+                <xacro:arg name="physical_params" default="$(find ur_description)/config/$(arg ur_type)/physical_parameters.yaml"/>
+                <xacro:arg name="visual_params" default="$(find ur_description)/config/$(arg ur_type)/visual_parameters.yaml"/>
+                <xacro:arg name="transmission_hw_interface" default=""/>
+                <xacro:arg name="safety_limits" default="false"/>
+                <xacro:arg name="safety_pos_margin" default="0.15"/>
+                <xacro:arg name="safety_k_position" default="20"/>
+                <!-- ros2_control related parameters -->
+                <xacro:arg name="headless_mode" default="false" />
+                <xacro:arg name="robot_ip" default="0.0.0.0" />
+                <xacro:arg name="script_filename" default=""/>
+                <xacro:arg name="output_recipe_filename" default=""/>
+                <xacro:arg name="input_recipe_filename" default=""/>
+                <xacro:arg name="reverse_ip" default="0.0.0.0"/>
+                <xacro:arg name="script_command_port" default="50004"/>
+                <xacro:arg name="reverse_port" default="50001"/>
+                <xacro:arg name="script_sender_port" default="50002"/>
+                <xacro:arg name="trajectory_port" default="50003"/>
+                <!--   tool communication related parameters-->
+                <xacro:arg name="use_tool_communication" default="false" />
+                <xacro:arg name="tool_voltage" default="0" />
+                <xacro:arg name="tool_parity" default="0" />
+                <xacro:arg name="tool_baud_rate" default="115200" />
+                <xacro:arg name="tool_stop_bits" default="1" />
+                <xacro:arg name="tool_rx_idle_chars" default="1.5" />
+                <xacro:arg name="tool_tx_idle_chars" default="3.5" />
+                <xacro:arg name="tool_device_name" default="/tmp/ttyUR" />
+                <xacro:arg name="tool_tcp_port" default="54321" />
+                    <!-- Simulation parameters -->
+                <xacro:arg name="use_fake_hardware" default="false" />
+                <xacro:arg name="fake_sensor_commands" default="false" />
+                <xacro:arg name="sim_gazebo" default="false" />
+                <xacro:arg name="sim_ignition" default="false" />
+                <xacro:arg name="simulation_controllers" default="" />
+                <!-- initial position for simulations (Fake Hardware, Gazebo, Ignition) -->
+                <xacro:arg name="initial_positions_file" default="$(find ur_description)/config/initial_positions.yaml"/>
+                <!-- convert to property to use substitution in function -->
+                <xacro:property name="initial_positions_file" default="$(arg initial_positions_file)"/>
+                <!-- arm -->
+                <xacro:ur_robot
+                    name="$(arg name)"
+                    tf_prefix="$(arg ur_prefix)"
+                    parent="${resolved_parent_link}"
+                    joint_limits_parameters_file="$(arg joint_limit_params)"
+                    kinematics_parameters_file="$(arg kinematics_params)"
+                    physical_parameters_file="$(arg physical_params)"
+                    visual_parameters_file="$(arg visual_params)"
+                    transmission_hw_interface="$(arg transmission_hw_interface)"
+                    safety_limits="$(arg safety_limits)"
+                    safety_pos_margin="$(arg safety_pos_margin)"
+                    safety_k_position="$(arg safety_k_position)"
+                    use_fake_hardware="$(arg use_fake_hardware)"
+                    fake_sensor_commands="$(arg fake_sensor_commands)"
+                    sim_gazebo="$(arg sim_gazebo)"
+                    sim_ignition="$(arg sim_ignition)"
+                    headless_mode="$(arg headless_mode)"
+                    initial_positions="${xacro.load_yaml(initial_positions_file)}"
+                    use_tool_communication="$(arg use_tool_communication)"
+                    tool_voltage="$(arg tool_voltage)"
+                    tool_parity="$(arg tool_parity)"
+                    tool_baud_rate="$(arg tool_baud_rate)"
+                    tool_stop_bits="$(arg tool_stop_bits)"
+                    tool_rx_idle_chars="$(arg tool_rx_idle_chars)"
+                    tool_tx_idle_chars="$(arg tool_tx_idle_chars)"
+                    tool_device_name="$(arg tool_device_name)"
+                    tool_tcp_port="$(arg tool_tcp_port)"
+                    robot_ip="$(arg robot_ip)"
+                    script_filename="$(arg script_filename)"
+                    output_recipe_filename="$(arg output_recipe_filename)"
+                    input_recipe_filename="$(arg input_recipe_filename)"
+                    reverse_ip="$(arg reverse_ip)"
+                    script_command_port="$(arg script_command_port)"
+                    reverse_port="$(arg reverse_port)"
+                    script_sender_port="$(arg script_sender_port)"
+                    trajectory_port="$(arg trajectory_port)"
+                    >
+                    <origin xyz="0 0 0" rpy="0 0 0" />          <!-- position robot in the world -->
+                </xacro:ur_robot>
             </xacro:if>
-            <xacro:unless value="${stack_qty == 1}">
-                <!-- <link name='${str(resolved_robot_part)}'/> -->
-                <!-- UR5e -->
-                <xacro:if value="${ str(resolved_robot_part) == 'ur5e' }">
-                    <xacro:include filename="$(find ur_description)/urdf/ur_macro.xacro"/>
-                    <xacro:arg name="ur_type" default='ur5e'/>
-                    <xacro:arg name="ur_prefix" default='$(arg ur_type)__'/>
-                    <xacro:arg name="joint_limit_params" default="$(find ur_description)/config/$(arg ur_type)/joint_limits.yaml"/>
-                    <xacro:arg name="kinematics_params" default="$(find ur_description)/config/$(arg ur_type)/default_kinematics.yaml"/>
-                    <xacro:arg name="physical_params" default="$(find ur_description)/config/$(arg ur_type)/physical_parameters.yaml"/>
-                    <xacro:arg name="visual_params" default="$(find ur_description)/config/$(arg ur_type)/visual_parameters.yaml"/>
-                    <xacro:arg name="transmission_hw_interface" default=""/>
-                    <xacro:arg name="safety_limits" default="false"/>
-                    <xacro:arg name="safety_pos_margin" default="0.15"/>
-                    <xacro:arg name="safety_k_position" default="20"/>
-                    <!-- ros2_control related parameters -->
-                    <xacro:arg name="headless_mode" default="false" />
-                    <xacro:arg name="robot_ip" default="0.0.0.0" />
-                    <xacro:arg name="script_filename" default=""/>
-                    <xacro:arg name="output_recipe_filename" default=""/>
-                    <xacro:arg name="input_recipe_filename" default=""/>
-                    <xacro:arg name="reverse_ip" default="0.0.0.0"/>
-                    <xacro:arg name="script_command_port" default="50004"/>
-                    <xacro:arg name="reverse_port" default="50001"/>
-                    <xacro:arg name="script_sender_port" default="50002"/>
-                    <xacro:arg name="trajectory_port" default="50003"/>
-                    <!--   tool communication related parameters-->
-                    <xacro:arg name="use_tool_communication" default="false" />
-                    <xacro:arg name="tool_voltage" default="0" />
-                    <xacro:arg name="tool_parity" default="0" />
-                    <xacro:arg name="tool_baud_rate" default="115200" />
-                    <xacro:arg name="tool_stop_bits" default="1" />
-                    <xacro:arg name="tool_rx_idle_chars" default="1.5" />
-                    <xacro:arg name="tool_tx_idle_chars" default="3.5" />
-                    <xacro:arg name="tool_device_name" default="/tmp/ttyUR" />
-                    <xacro:arg name="tool_tcp_port" default="54321" />
-                        <!-- Simulation parameters -->
-                    <xacro:arg name="use_fake_hardware" default="false" />
-                    <xacro:arg name="fake_sensor_commands" default="false" />
-                    <xacro:arg name="sim_gazebo" default="false" />
-                    <xacro:arg name="sim_ignition" default="false" />
-                    <xacro:arg name="simulation_controllers" default="" />
-                    <!-- initial position for simulations (Fake Hardware, Gazebo, Ignition) -->
-                    <xacro:arg name="initial_positions_file" default="$(find ur_description)/config/initial_positions.yaml"/>
-                    <!-- convert to property to use substitution in function -->
-                    <xacro:property name="initial_positions_file" default="$(arg initial_positions_file)"/>
-                    <!-- arm -->
-                    <xacro:ur_robot
-                        name="$(arg name)"
-                        tf_prefix="$(arg ur_prefix)"
-                        parent="${resolved_parent_part}"
-                        joint_limits_parameters_file="$(arg joint_limit_params)"
-                        kinematics_parameters_file="$(arg kinematics_params)"
-                        physical_parameters_file="$(arg physical_params)"
-                        visual_parameters_file="$(arg visual_params)"
-                        transmission_hw_interface="$(arg transmission_hw_interface)"
-                        safety_limits="$(arg safety_limits)"
-                        safety_pos_margin="$(arg safety_pos_margin)"
-                        safety_k_position="$(arg safety_k_position)"
-                        use_fake_hardware="$(arg use_fake_hardware)"
-                        fake_sensor_commands="$(arg fake_sensor_commands)"
-                        sim_gazebo="$(arg sim_gazebo)"
-                        sim_ignition="$(arg sim_ignition)"
-                        headless_mode="$(arg headless_mode)"
-                        initial_positions="${xacro.load_yaml(initial_positions_file)}"
-                        use_tool_communication="$(arg use_tool_communication)"
-                        tool_voltage="$(arg tool_voltage)"
-                        tool_parity="$(arg tool_parity)"
-                        tool_baud_rate="$(arg tool_baud_rate)"
-                        tool_stop_bits="$(arg tool_stop_bits)"
-                        tool_rx_idle_chars="$(arg tool_rx_idle_chars)"
-                        tool_tx_idle_chars="$(arg tool_tx_idle_chars)"
-                        tool_device_name="$(arg tool_device_name)"
-                        tool_tcp_port="$(arg tool_tcp_port)"
-                        robot_ip="$(arg robot_ip)"
-                        script_filename="$(arg script_filename)"
-                        output_recipe_filename="$(arg output_recipe_filename)"
-                        input_recipe_filename="$(arg input_recipe_filename)"
-                        reverse_ip="$(arg reverse_ip)"
-                        script_command_port="$(arg script_command_port)"
-                        reverse_port="$(arg reverse_port)"
-                        script_sender_port="$(arg script_sender_port)"
-                        trajectory_port="$(arg trajectory_port)"
-                        >
-                        <origin xyz="0 0 0" rpy="0 0 0" />          <!-- position robot in the world -->
-                    </xacro:ur_robot>
-                </xacro:if>
-                <!-- Robot cart -->
-                <xacro:if value="${ str(resolved_robot_part) == 'cart' }">
-                    <xacro:include filename="../../base_mounts/cart/cart_macro.urdf.xacro"/>
-                    <xacro:cart_macro
-                        cart_prefix="cart__"
-                        cart_parent="$(arg parent${stack_qty - 1})"
-                    />
-                </xacro:if>
-                <!-- <link name="$(arg robot_part${stack_qty - 1})" /> -->
-            </xacro:unless>
+            <!-- Robot cart -->
+            <xacro:if value="${ str(resolved_part) == 'cart' }">
+                <xacro:include filename="$(arg urdf_base_path)/base_mounts/cart/macro/cart_macro.urdf.xacro"/>
+                <xacro:cart_macro
+                    cart_prefix="cart__"
+                    cart_parent="${resolved_parent_part}"
+                    mesh_base_path="$(arg mesh_base_path)"
+                />
+            </xacro:if>
+            <xacro:if value="${ str(resolved_part) == 'mock_pruner' }">
+                <xacro:include filename="$(arg urdf_base_path)/end_effectors/mock_pruner/macro/mock_pruner_macro.urdf.xacro"/>
+                <!-- Args -->
+                <xacro:arg name="mock_pruner_prefix" default="mock_pruner__" />
+                <xacro:arg name="mesh_base_path" default="" />
+                <xacro:arg name="tof0_offset_x" default="0.02" />
+                <xacro:arg name="tof1_offset_x" default="-0.02" />
+                <!-- mock_pruner macro -->
+                <!-- <xacro:include filename="./macro/mock_pruner_macro.urdf.xacro" /> -->
+                <xacro:mock_pruner_macro
+                    eef_prefix="$(arg mock_pruner_prefix)"
+                    parent_link="${resolved_parent_link}"
+                    mesh_base_path="$(arg mesh_base_path)"
+                    tof0_offset='$(arg tof0_offset_x)'
+                    tof1_offset='$(arg tof1_offset_x)'
+                    camera_offset=''
+                />
+            </xacro:if>
+            <!-- <link name="$(arg robot_part${stack_qty - 1})" /> -->
+            <!-- </xacro:unless> -->
             <!-- call macro recursively -->
             <xacro:main_loop stack_qty="${stack_qty - 1}"/>
