Commit message: added dynamic building of the urdf. needs testing

File: pybullet_tree_sim/urdf/tmp/robot.urdf (robot description, URDF)
Before this commit: robot pruning_robot, 3 links, 3 joints
Links:
- removed link mock_pruner
- removed link ur5e
- added link cart__base
- added link cart__cart, mass 20.0; collision box size=0.5 0.5 0.75711; visual mesh filename=/home/luke/dev/pybullet/pybullet-tree-sim/pybullet_tree_sim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
- added link cart__tool0
- added link mock_pruner__base, mass 2.0; collision mesh filename=/home/luke/dev/pybullet/pybullet-tree-sim/pybullet_tree_sim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; visual mesh filename=/home/luke/dev/pybullet/pybullet-tree-sim/pybullet_tree_sim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
- added link mock_pruner__camera0
- added link mock_pruner__tof0
- added link mock_pruner__tof1
- added link mock_pruner__tool0
- added link ur5e__base
- added link ur5e__base_link
- added link ur5e__base_link_inertia, mass 4.0; collision mesh filename=package://ur_description/meshes/ur5e/collision/base.stl; visual mesh filename=package://ur_description/meshes/ur5e/visual/base.dae
- added link ur5e__flange
- added link ur5e__forearm_link, mass 2.846; collision mesh filename=package://ur_description/meshes/ur5e/collision/forearm.stl; visual mesh filename=package://ur_description/meshes/ur5e/visual/forearm.dae
- added link ur5e__ft_frame
- added link ur5e__shoulder_link, mass 3.761; collision mesh filename=package://ur_description/meshes/ur5e/collision/shoulder.stl; visual mesh filename=package://ur_description/meshes/ur5e/visual/shoulder.dae
- added link ur5e__tool0
- added link ur5e__upper_arm_link, mass 8.058; collision mesh filename=package://ur_description/meshes/ur5e/collision/upperarm.stl; visual mesh filename=package://ur_description/meshes/ur5e/visual/upperarm.dae
- added link ur5e__wrist_1_link, mass 1.37; collision mesh filename=package://ur_description/meshes/ur5e/collision/wrist1.stl; visual mesh filename=package://ur_description/meshes/ur5e/visual/wrist1.dae
- added link ur5e__wrist_2_link, mass 1.3; collision mesh filename=package://ur_description/meshes/ur5e/collision/wrist2.stl; visual mesh filename=package://ur_description/meshes/ur5e/visual/wrist2.dae
- added link ur5e__wrist_3_link, mass 0.365; collision mesh filename=package://ur_description/meshes/ur5e/collision/wrist3.stl; visual mesh filename=package://ur_description/meshes/ur5e/visual/wrist3.dae
Joints:
- removed joint mock_pruner--ur5e
- removed joint ur5e--cart
- removed joint world--link-1
- added joint cart__base--cart__cart: type fixed, parent cart__base, child cart__cart, origin xyz=0 0 0 rpy=0 0 0
- added joint cart__cart--cart__tool0: type fixed, parent cart__cart, child cart__tool0, origin xyz=0 0 0.75711 rpy=0 0 0
- added joint mock_pruner__base--camera0: type fixed, parent mock_pruner__base, child mock_pruner__camera0, origin xyz=0 0 0 rpy=0 0 0
- added joint mock_pruner__base--tof0: type fixed, parent mock_pruner__base, child mock_pruner__tof0, origin xyz=0.02 0 0 rpy=0 0 0
- added joint mock_pruner__base--tof1: type fixed, parent mock_pruner__base, child mock_pruner__tof1, origin xyz=-0.02 0 0 rpy=0 0 0
- added joint mock_pruner__base--tool0: type fixed, parent mock_pruner__base, child mock_pruner__tool0, origin xyz=0 0 0 rpy=0 0 0
- added joint ur5e__base_joint: type fixed, parent cart__tool0, child ur5e__base_link, origin xyz=0 0 0 rpy=0 0 0
- added joint ur5e__base_link-base_fixed_joint: type fixed, parent ur5e__base_link, child ur5e__base, origin xyz=0 0 0 rpy=0 0 3.141592653589793
- added joint ur5e__base_link-base_link_inertia: type fixed, parent ur5e__base_link, child ur5e__base_link_inertia, origin xyz=0 0 0 rpy=0 0 3.141592653589793
- added joint ur5e__elbow_joint: type revolute, parent ur5e__upper_arm_link, child ur5e__forearm_link, origin xyz=-0.425 0 0 rpy=0 0 0, axis 0 0 1, limit lower=-3.141592653589793 upper=3.141592653589793 effort=150.0 velocity=3.141592653589793
- added joint ur5e__flange-tool0: type fixed, parent ur5e__flange, child ur5e__tool0, origin xyz=0 0 0 rpy=1.5707963267948966 0 1.5707963267948966
- added joint ur5e__shoulder_lift_joint: type revolute, parent ur5e__shoulder_link, child ur5e__upper_arm_link, origin xyz=0 0 0 rpy=1.570796327 0 0, axis 0 0 1, limit lower=-6.283185307179586 upper=6.283185307179586 effort=150.0 velocity=3.141592653589793
- added joint ur5e__shoulder_pan_joint: type revolute, parent ur5e__base_link_inertia, child ur5e__shoulder_link, origin xyz=0 0 0.1625 rpy=0 0 0, axis 0 0 1, limit lower=-6.283185307179586 upper=6.283185307179586 effort=150.0 velocity=3.141592653589793
- added joint ur5e__tool0--mock_pruner__base: type fixed, parent ur5e__tool0, child mock_pruner__base, origin xyz=0 0 0 rpy=0 0 0
- added joint ur5e__wrist_1_joint: type revolute, parent ur5e__forearm_link, child ur5e__wrist_1_link, origin xyz=-0.3922 0 0.1333 rpy=0 0 0, axis 0 0 1, limit lower=-6.283185307179586 upper=6.283185307179586 effort=28.0 velocity=3.141592653589793
- added joint ur5e__wrist_2_joint: type revolute, parent ur5e__wrist_1_link, child ur5e__wrist_2_link, origin xyz=0 -0.0997 -2.044881182297852e-11 rpy=1.570796327 0 0, axis 0 0 1, limit lower=-6.283185307179586 upper=6.283185307179586 effort=28.0 velocity=3.141592653589793
- added joint ur5e__wrist_3-flange: type fixed, parent ur5e__wrist_3_link, child ur5e__flange, origin xyz=0 0 0 rpy=0 -1.5707963267948966 -1.5707963267948966
- added joint ur5e__wrist_3_joint: type revolute, parent ur5e__wrist_2_link, child ur5e__wrist_3_link, origin xyz=0 0.0996 -2.042830148012698e-11 rpy=1.570796326589793 3.141592653589793 3.141592653589793, axis 0 0 1, limit lower=-6.283185307179586 upper=6.283185307179586 effort=28.0 velocity=3.141592653589793
- added joint ur5e__wrist_3_link-ft_frame: type fixed, parent ur5e__wrist_3_link, child ur5e__ft_frame, origin xyz=0 0 0 rpy=3.141592653589793 0 0
- added joint world--cart__base: type fixed, parent world, child cart__base, origin xyz=0 0 0 rpy=0 0 0

Commit message: successfully reading and plotting tof0 and tof1 from mock pruner

File: pybullet_tree_sim/urdf/end_effectors/mock_pruner/macro/mock_pruner_macro.urdf.xacro (robot description, xacro)
@@ -9,8 +9,14 @@
         <!-- static properties -->
         <xacro:property name="mock_pruner_mass" value="2.0" />
+        <xacro:property name="base__tool0_offset" value="0.0 0.0 0.27208"/>
+        <xacro:property name="base__tof0_offset" value="${tof0_offset} 0 0.142"/>
+        <xacro:property name="base__tof1_offset" value="${tof1_offset} 0 0.142"/>
+        <!-- <xacro:property name="base__tof0_offset" value="${tof0_offset} 0 0.15"/> -->
+        <!-- <xacro:property name="base__tof1_offset" value="${tof1_offset} 0 0.15"/> -->
+        <xacro:property name="base__camera0_offset" value="0.0 0.0600 0.19094"/>
         <!-- additional args -->
         <xacro:arg name="dovetail_male_mount_prefix" default="dovetail_male_mount__" />
         <xacro:arg name="dovetail_female_mount_prefix" default="dovetail_female_mount__" />
-        <xacro:arg name="mesh_base_path" default="" />
+        <xacro:arg name="mesh_base_path" default=""/>
         <xacro:arg name="urdf_base_path" default=""/>
         <!-- dovetail_mount macro -->
@@ -66,5 +72,5 @@
         </joint>
         <joint name="${eef_prefix}base--camera0" type="fixed">
-            <origin xyz="0 0 0" rpy="0 0 0"/>
+            <origin xyz="${base__camera0_offset}" rpy="0 0 0"/>
             <parent link="${eef_prefix}base" />
             <child link="${eef_prefix}camera0" />
@@ -72,15 +78,15 @@
         <joint name="${eef_prefix}base--tof0" type="fixed">
             <!-- <xacro:insert_block name="origin"/> -->
-            <origin xyz="${tof0_offset} 0 0" rpy="0 0 0"/>
+            <origin xyz="${base__tof0_offset}" rpy="0 0 0"/>
             <parent link="${eef_prefix}base" />
             <child link="${eef_prefix}tof0" />
         </joint>
         <joint name="${eef_prefix}base--tof1" type="fixed">
-            <origin xyz="${tof1_offset} 0 0" rpy="0 0 0"/>
+            <origin xyz="${base__tof1_offset}" rpy="0 0 0"/>
             <parent link="${eef_prefix}base" />
             <child link="${eef_prefix}tof1" />
         </joint>
         <joint name="${eef_prefix}base--tool0" type="fixed">
-            <origin xyz="0 0 0" rpy="0 0 0"/>
+            <origin xyz="${base__tool0_offset}" rpy="0 0 0"/>
             <parent link="${eef_prefix}base" />
             <child link="${eef_prefix}tool0" />

File: pybullet_tree_sim/urdf/shapes/cylinder/cylinder.urdf (robot description, URDF)
Before this commit: robot cylinder, 2 links, 1 joints
Links:
- link cylinder: geometry collision cylinder length=2.85 radius=0.0508; visual cylinder length=2.85 radius=0.0508

File: pybullet_tree_sim/urdf/tmp/robot.urdf (robot description, URDF)
Before this commit: robot pruning_robot, 27 links, 26 joints
Joints:
- joint mock_pruner__base--camera0: origin xyz=0 0 0 rpy=0 0 0 -> xyz=0.0 0.0600 0.19094 rpy=0 0 0
- joint mock_pruner__base--tof0: origin xyz=0.02 0 0 rpy=0 0 0 -> xyz=0.1 0 0.142 rpy=0 0 0
- joint mock_pruner__base--tof1: origin xyz=-0.02 0 0 rpy=0 0 0 -> xyz=-0.1 0 0.142 rpy=0 0 0
- joint mock_pruner__base--tool0: origin xyz=0 0 0 rpy=0 0 0 -> xyz=0.0 0.0 0.27208 rpy=0 0 0

Commit message: fixed depth linearization

File: pybullet_tree_sim/urdf/end_effectors/mock_pruner/macro/mock_pruner_macro.urdf.xacro (robot description, xacro)
@@ -10,4 +10,5 @@
         <xacro:property name="mock_pruner_mass" value="2.0" />
         <xacro:property name="base__tool0_offset" value="0.0 0.0 0.27208"/>
+        <!-- <xacro:property name="base__tool0_offset" value="0.0 0.0 0.20"/> -->
         <xacro:property name="base__tof0_offset" value="${tof0_offset} 0 0.142"/>
         <xacro:property name="base__tof1_offset" value="${tof1_offset} 0 0.142"/>

File: pybullet_tree_sim/urdf/shapes/cylinder/cylinder.urdf (robot description, URDF)
Before this commit: robot cylinder, 2 links, 1 joints
Links:
- link cylinder: geometry collision cylinder length=2.82 radius=0.0254; visual cylinder length=2.82 radius=0.0254
