Commit message: working base robot class for final approach controller

File: pybullet_tree_sim/urdf/end_effectors/dovetail_mount/macro/dovetail_mount_macro.urdf.xacro (robot description, xacro)
@@ -3,4 +3,5 @@
     <xacro:property name="dovetail_male_tool0_height" value="0.008"/>
     <xacro:property name="dovetail_female_tool0_height" value="0.023"/>
+    <xacro:property name="dovetail_male_rot_offset" value="0.0 0.0 0.0"/>
     <xacro:macro name="dovetail_male_mount_macro" params="parent_link dovetail_male_mount_prefix mesh_base_path">
         <!-- ==================== -->
@@ -36,5 +37,5 @@
         <!-- joints -->
         <joint name="${parent_link}--${dovetail_male_mount_prefix}base" type="fixed">
-            <origin xyz="0 0 0" rpy="0 0 0"/>
+            <origin xyz="0 0 0" rpy="${dovetail_male_rot_offset}"/>
             <parent link="${parent_link}"/>
             <child link="${dovetail_male_mount_prefix}base"/>

File: pybullet_tree_sim/urdf/robot/generic/robot.urdf.xacro (robot description, xacro)
@@ -26,5 +26,5 @@
                 <xacro:property name='resolved_parent_link' value='world'/>
             </xacro:if>
-            <xacro:unless value="${ str(resolved_parent_part) == 'world'}">
+            <xacro:unless value="${ str(resolved_parent_part) == 'world' }">
                 <xacro:property name='resolved_parent_link' value="${resolved_parent_part}__tool0"/>
             </xacro:unless>
@@ -147,4 +147,5 @@
         </xacro:if>
     </xacro:macro>
+    <!-- call main loop -->
     <xacro:main_loop stack_qty="$(arg robot_stack_qty)"/>
 </robot>

File: pybullet_tree_sim/urdf/shapes/cylinder/cylinder.urdf (robot description, URDF)
Before this commit: robot cylinder, 2 links, 1 joints
Links:
- link cylinder: geometry collision cylinder length=2.81 radius=0.0127; visual cylinder length=2.81 radius=0.0127

File: pybullet_tree_sim/urdf/tmp/robot.urdf (robot description, URDF)
Before this commit: robot pruning_robot, 27 links, 26 joints
Joints:
- joint ur5e__tool0--dovetail_male_mount__base: origin xyz=0 0 0 rpy=0 0 0 -> xyz=0 0 0 rpy=0.0 0.0 0.0
