Commit message: added dovetail mount, modified mock pruner

File: pybullet_tree_sim/urdf/base_mounts/cart/macro/cart_macro.urdf.xacro (robot description, xacro)
@@ -28,5 +28,5 @@
         </visual>
         <collision>
-            <origin rpy="0.0 0.0 0.0" xyz="0.0 0.0 -0.3786"/>
+            <origin rpy="0.0 0.0 0.0" xyz="0.0 0.0 0.0"/>
             <geometry>
                 <box size="${cart_collision_box_x} ${cart_collision_box_y} ${cart_collision_box_z}"/>

File: pybullet_tree_sim/urdf/end_effectors/mock_pruner/macro/mock_pruner_macro.urdf.xacro (robot description, xacro)
@@ -2,9 +2,9 @@
 <robot xmlns:xacro="https://ros.org/wiki/xacro" name="mock_pruner">
     <!-- Mock Pruner -->
-    <xacro:arg name="name" default="mock_pruner"/>
+    <!-- <xacro:arg name="name" default="mock_pruner"/> -->
     <!-- <xacro:arg name="mesh_base_path" default="./"/> -->
     <!-- <xacro:property name="end_effector_parent" value="" /> -->
     <!-- Materials -->
-    <xacro:macro name="mock_pruner_macro" params="parent_link eef_prefix tof0_offset tof1_offset camera_offset mesh_base_path">
+    <xacro:macro name="mock_pruner_macro" params="parent_link eef_prefix tof0_offset tof1_offset camera_offset mesh_base_path urdf_base_path">
         <!-- ================== -->
         <!--     Properties     -->
@@ -14,4 +14,17 @@
         <!--       Links        -->
         <!-- ================== -->
+        <!-- parent_link dovetail_male_mount_prefix mesh_base_path -->
+        <xacro:arg name="dovetail_male_mount_prefix" default="dovetail_male_mount__" />
+        <xacro:arg name="dovetail_female_mount_prefix" default="dovetail_female_mount__" />
+        <xacro:arg name="mesh_base_path" default="" />
+        <xacro:arg name="urdf_base_path" default=""/>
+        <!-- dovetail_mount macro -->
+        <xacro:include filename="${urdf_base_path}/end_effectors/dovetail_mount/macro/dovetail_mount_macro.urdf.xacro" />
+        <xacro:dovetail_mount_macro
+            parent_link="${parent_link}"
+            dovetail_male_mount_prefix="$(arg dovetail_male_mount_prefix)"
+            dovetail_female_mount_prefix="$(arg dovetail_female_mount_prefix)"
+            mesh_base_path="${mesh_base_path}"
+        />
         <link name="${eef_prefix}base" >
             <visual>
@@ -21,5 +34,5 @@
                 <origin xyz="0 0 0" rpy="0 0 0"/>
                 <geometry>
-                    <mesh filename="${mesh_base_path}/end_effectors/mock_pruner/MockPrunerASSEMBLED.STL" />
+                    <mesh filename="${mesh_base_path}/end_effectors/mock_pruner/MockPruner.STL" />
                 </geometry>
             </visual>
@@ -27,5 +40,5 @@
                 <origin xyz="0 0 0" rpy="0 0 0"/>
                 <geometry>
-                    <mesh filename="${mesh_base_path}/end_effectors/mock_pruner/MockPrunerASSEMBLED.STL" />
+                    <mesh filename="${mesh_base_path}/end_effectors/mock_pruner/MockPruner.STL" />
                 </geometry>
             </collision>
@@ -46,7 +59,7 @@
         <!--     Joints        -->
         <!-- ================== -->
-        <joint name="${parent_link}--${eef_prefix}base" type="fixed">
+        <joint name="$(arg dovetail_female_mount_prefix)tool0--${eef_prefix}base" type="fixed">
             <origin xyz="0 0 0" rpy="0 0 0"/>
-            <parent link="${parent_link}"/>
+            <parent link="$(arg dovetail_female_mount_prefix)tool0"/>
             <child link="${eef_prefix}base"/>
         </joint>

File: pybullet_tree_sim/urdf/robot/generic/robot.urdf.xacro (robot description, xacro)
@@ -23,8 +23,10 @@
             <xacro:property name='resolved_part_base' value="${resolved_part}__base}"/>
             <xacro:property name='resolved_parent_part' value="$(arg parent${stack_qty - 1})"/>
-            <xacro:property name='resolved_parent_link' value="${resolved_parent_part}__tool0"/>
-            <!-- <xacro:unless value="${stack_qty == 1}"> -->
-            <!-- <link name="${resolved_part}"/> -->
-            <!-- <link name='${str(resolved_robot_part)}'/> -->
+            <xacro:if value="${ str(resolved_parent_part) == 'world'}">
+                <xacro:property name='resolved_parent_link' value='world'/>
+            </xacro:if>
+            <xacro:unless value="${ str(resolved_parent_part) == 'world'}">
+                <xacro:property name='resolved_parent_link' value="${resolved_parent_part}__tool0"/>
+            </xacro:unless>
             <!-- UR5e -->
             <xacro:if value="${ str(resolved_part) == 'ur5e' }">
@@ -128,10 +130,10 @@
                 <xacro:arg name="tof0_offset_x" default="0.02" />
                 <xacro:arg name="tof1_offset_x" default="-0.02" />
-                <!-- mock_pruner macro -->
-                <!-- <xacro:include filename="./macro/mock_pruner_macro.urdf.xacro" /> -->
+                <!-- mock_pruner  -->
                 <xacro:mock_pruner_macro
                     eef_prefix="$(arg mock_pruner_prefix)"
                     parent_link="${resolved_parent_link}"
                     mesh_base_path="$(arg mesh_base_path)"
+                    urdf_base_path="$(arg urdf_base_path)"
                     tof0_offset='$(arg tof0_offset_x)'
                     tof1_offset='$(arg tof1_offset_x)'

File: pybullet_tree_sim/urdf/tmp/robot.urdf (robot description, URDF)
Before this commit: robot pruning_robot, 21 links, 20 joints
Links:
- added link dovetail_female_mount__base
- added link dovetail_female_mount__body, mass 0.025; collision mesh filename=/home/luke/dev/pybullet/pybullet-tree-sim/pybullet_tree_sim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; visual mesh filename=/home/luke/dev/pybullet/pybullet-tree-sim/pybullet_tree_sim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
- added link dovetail_female_mount__tool0
- added link dovetail_male_mount__base
- added link dovetail_male_mount__body, mass 0.025; collision mesh filename=/home/luke/dev/pybullet/pybullet-tree-sim/pybullet_tree_sim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; visual mesh filename=/home/luke/dev/pybullet/pybullet-tree-sim/pybullet_tree_sim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
- added link dovetail_male_mount__tool0
- link ur5e__base_link_inertia: geometry collision mesh filename=/opt/ros/humble/share/ur_description/meshes/ur5e/collision/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; visual mesh filename=/opt/ros/humble/share/ur_description/meshes/ur5e/visual/bas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
- link ur5e__forearm_link: geometry collision mesh filename=/opt/ros/humble/share/ur_description/meshes/ur5e/collision/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; visual mesh filename=/opt/ros/humble/share/ur_description/meshes/ur5e/visual/for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
- link ur5e__shoulder_link: geometry collision mesh filename=/opt/ros/humble/share/ur_description/meshes/ur5e/collision/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; visual mesh filename=/opt/ros/humble/share/ur_description/meshes/ur5e/visual/sho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
- link ur5e__upper_arm_link: geometry collision mesh filename=/opt/ros/humble/share/ur_description/meshes/ur5e/collision/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; visual mesh filename=/opt/ros/humble/share/ur_description/meshes/ur5e/visual/upp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
- link ur5e__wrist_1_link: geometry collision mesh filename=/opt/ros/humble/share/ur_description/meshes/ur5e/collision/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; visual mesh filename=/opt/ros/humble/share/ur_description/meshes/ur5e/visual/wri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
- link ur5e__wrist_2_link: geometry collision mesh filename=/opt/ros/humble/share/ur_description/meshes/ur5e/collision/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; visual mesh filename=/opt/ros/humble/share/ur_description/meshes/ur5e/visual/wri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
- link ur5e__wrist_3_link: geometry collision mesh filename=/opt/ros/humble/share/ur_description/meshes/ur5e/collision/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; visual mesh filename=/opt/ros/humble/share/ur_description/meshes/ur5e/visual/wri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
Joints:
- removed joint ur5e__tool0--mock_pruner__base
- added joint dovetail_female_mount__base--body: type fixed, parent dovetail_female_mount__base, child dovetail_female_mount__body, origin xyz=0 0 0 rpy=0 0 0
- added joint dovetail_female_mount__body--tool0: type fixed, parent dovetail_female_mount__body, child dovetail_female_mount__tool0, origin xyz=0 0 0 rpy=0 0 0
- added joint dovetail_female_mount__tool0--mock_pruner__base: type fixed, parent dovetail_female_mount__tool0, child mock_pruner__base, origin xyz=0 0 0 rpy=0 0 0
- added joint dovetail_male_mount__base--body: type fixed, parent dovetail_male_mount__base, child dovetail_male_mount__body, origin xyz=0 0 0 rpy=0 0 0
- added joint dovetail_male_mount__body--tool0: type fixed, parent dovetail_male_mount__body, child dovetail_male_mount__tool0, origin xyz=0 0 0.008 rpy=0 0 0
- added joint dovetail_male_mount__tool0--dovetail_female_mount__base: type fixed, parent dovetail_male_mount__tool0, child dovetail_female_mount__base, origin xyz=0 0 0.023 rpy=0 0 0
- added joint ur5e__tool0--dovetail_male_mount__base: type fixed, parent ur5e__tool0, child dovetail_male_mount__base, origin xyz=0 0 0 rpy=0 0 0

Commit message: current updates for cindy code review

File: pybullet_tree_sim/urdf/base_mounts/cart/macro/cart_macro.urdf.xacro (robot description, xacro)
@@ -3,12 +3,9 @@
 <xacro:macro name="cart_macro" params="cart_prefix:='cart__' cart_parent:='world' mesh_base_path">
     <!-- ================== -->
-    <!--     Materials      -->
+    <!--     Cart Maacro    -->
     <!-- ================== -->
     <material name="LightGrey">
         <color rgba="0.7 0.7 0.7 1.0"/>
     </material>
-    <!-- ================== -->
-    <!--     Properties     -->
-    <!-- ================== -->
     <xacro:property name="cart_mass" value="20.0"/>
     <xacro:property name="cart_collision_box_x" value='0.5'/>
@@ -21,5 +18,5 @@
     <link name="${cart_prefix}cart">
         <visual>
-            <origin rpy="0.0 0.0 0.0" xyz="0.0 0.0 0.0"/>
+            <origin rpy="0.0 0.0 0.0" xyz="0.0 0.0 ${cart_collision_box_z}"/>
             <geometry>
                 <mesh filename="${mesh_base_path}/base_mounts/cart/cart.obj"/>
@@ -28,5 +25,5 @@
         </visual>
         <collision>
-            <origin rpy="0.0 0.0 0.0" xyz="0.0 0.0 0.0"/>
+            <origin rpy="0.0 0.0 0.0" xyz="0.0 0.0 -${cart_collision_box_z / 2}"/>
             <geometry>
                 <box size="${cart_collision_box_x} ${cart_collision_box_y} ${cart_collision_box_z}"/>

File: pybullet_tree_sim/urdf/end_effectors/dovetail_mount/macro/dovetail_mount_macro.urdf.xacro (robot description, xacro)
@@ -100,4 +100,7 @@
     </xacro:macro>
     <xacro:macro name="dovetail_mount_macro" params="parent_link dovetail_male_mount_prefix dovetail_female_mount_prefix mesh_base_path">
+        <!-- =================== -->
+        <!--   Dovetail Mount    -->
+        <!-- =================== -->
         <xacro:dovetail_male_mount_macro
             parent_link="${parent_link}"

File: pybullet_tree_sim/urdf/end_effectors/mock_pruner/macro/mock_pruner_macro.urdf.xacro (robot description, xacro)
@@ -7,12 +7,7 @@
     <!-- Materials -->
     <xacro:macro name="mock_pruner_macro" params="parent_link eef_prefix tof0_offset tof1_offset camera_offset mesh_base_path urdf_base_path">
-        <!-- ================== -->
-        <!--     Properties     -->
-        <!-- ================== -->
+        <!-- static properties -->
         <xacro:property name="mock_pruner_mass" value="2.0" />
-        <!-- ================== -->
-        <!--       Links        -->
-        <!-- ================== -->
-        <!-- parent_link dovetail_male_mount_prefix mesh_base_path -->
+        <!-- additional args -->
         <xacro:arg name="dovetail_male_mount_prefix" default="dovetail_male_mount__" />
         <xacro:arg name="dovetail_female_mount_prefix" default="dovetail_female_mount__" />
@@ -27,4 +22,10 @@
             mesh_base_path="${mesh_base_path}"
         />
+        <!-- ==================== -->
+        <!--  Mock Pruner Macro   -->
+        <!-- ==================== -->
+        <!-- ================== -->
+        <!--       Links        -->
+        <!-- ================== -->
         <link name="${eef_prefix}base" >
             <visual>

Commit message: fixed cart collision box

File: pybullet_tree_sim/urdf/base_mounts/cart/macro/cart_macro.urdf.xacro (robot description, xacro)
@@ -10,5 +10,5 @@
     <xacro:property name="cart_mass" value="20.0"/>
     <xacro:property name="cart_collision_box_x" value='0.5'/>
-    <xacro:property name="cart_collision_box_y" value='0.5'/>
+    <xacro:property name="cart_collision_box_y" value='1.0'/>
     <xacro:property name="cart_collision_box_z" value='0.75711'/>
     <!-- ================== -->
@@ -25,5 +25,5 @@
         </visual>
         <collision>
-            <origin rpy="0.0 0.0 0.0" xyz="0.0 0.0 -${cart_collision_box_z / 2}"/>
+            <origin rpy="0.0 0.0 0.0" xyz="0.0 0.0 ${cart_collision_box_z / 2}"/>
             <geometry>
                 <box size="${cart_collision_box_x} ${cart_collision_box_y} ${cart_collision_box_z}"/>

File: pybullet_tree_sim/urdf/tmp/robot.urdf (robot description, URDF)
Before this commit: robot pruning_robot, 27 links, 26 joints
Links:
- link cart__cart: geometry collision box size=0.5 1.0 0.75711; visual mesh filename=/home/luke/dev/pybullet/pybullet-tree-sim/pybullet_tree_sim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
