Commit message: updated robot description from ROS2 implementations

File: pybullet_tree_sim/urdf/base_mounts/cart/macro/cart_macro.urdf.xacro (robot description, xacro)
@@ -12,4 +12,5 @@
     <xacro:property name="cart_collision_box_y" value='1.0'/>
     <xacro:property name="cart_collision_box_z" value='0.75711'/>
+    <xacro:property name="cart_tool0_mount_rotation" value="0.0 0.0 -${pi/4}"/>
     <!-- ================== -->
     <!--       Links        -->
@@ -20,5 +21,5 @@
             <origin rpy="0.0 0.0 0.0" xyz="0.0 0.0 ${cart_collision_box_z}"/>
             <geometry>
-                <mesh filename="${mesh_base_path}/base_mounts/cart/cart.obj"/>
+                <mesh filename="file://$(find branch_detection_system_description)/meshes/base_mounts/cart/cart.obj"/>
             </geometry>
             <material name="LightGrey"/>
@@ -44,5 +45,5 @@
     <link name="${cart_prefix}tool0"/>
     <!-- ================== -->
-    <!--     Joints        -->
+    <!--       Joints       -->
     <!-- ================== -->
     <joint name="${cart_parent}--${cart_prefix}base" type="fixed">
@@ -57,5 +58,5 @@
     </joint>
     <joint name="${cart_prefix}cart--${cart_prefix}tool0" type="fixed">
-        <origin rpy="0 0 0" xyz="0 0 ${cart_collision_box_z}"/>
+        <origin rpy="${cart_tool0_mount_rotation}" xyz="0 0 ${cart_collision_box_z}"/>
         <parent link="${cart_prefix}cart"/>
         <child link="${cart_prefix}tool0"/>

File: pybullet_tree_sim/urdf/end_effectors/dovetail_mount/macro/dovetail_mount_macro.urdf.xacro (robot description, xacro)
@@ -1,7 +1,4 @@
 <?xml version="1.0"?>
 <robot xmlns:xacro="https://ros.org/wiki/xacro" name="dovetail_mount">
-    <xacro:property name="dovetail_male_tool0_height" value="0.008"/>
-    <xacro:property name="dovetail_female_tool0_height" value="0.023"/>
-    <xacro:property name="dovetail_male_rot_offset" value="0.0 0.0 0.0"/>
     <xacro:macro name="dovetail_male_mount_macro" params="parent_link dovetail_male_mount_prefix mesh_base_path">
         <!-- ==================== -->
@@ -11,5 +8,7 @@
             <color rgba="0.749 0.580 0.894 1"/>
         </material>
-        <xacro:property name="dovetail_male_mass" value="0.025"/>
+        <xacro:property name="dovetail_male_mass" value="0.033"/>
+        <xacro:property name="dovetail_male_tool0_height" value="0.02293"/>
+        <xacro:property name="dovetail_male_rot_offset" value="0.0 0.0 0.0"/>
         <!-- links -->
         <link name="${dovetail_male_mount_prefix}base"/>
@@ -59,5 +58,7 @@
             <color rgba="0.929 0.710 0.145 1"/>
         </material>
-        <xacro:property name="dovetail_female_mass" value="0.025"/>
+        <xacro:property name="dovetail_female_mass" value="0.038"/>
+        <xacro:property name="dovetail_female_tool0_height" value="0.008"/>
+        <xacro:property name="dovetail_female_rot_offset" value="0.0 0.0 0.0"/>
         <!-- links -->
         <link name="${dovetail_female_mount_prefix}base"/>
@@ -85,5 +86,5 @@
         <!-- joints -->
         <joint name="${parent_link}--${dovetail_female_mount_prefix}base" type="fixed">
-            <origin xyz="0 0 ${dovetail_female_tool0_height}" rpy="0 0 0"/>
+            <origin xyz="0 0 0.0" rpy="${dovetail_female_rot_offset}"/>
             <parent link="${parent_link}"/>
             <child link="${dovetail_female_mount_prefix}base"/>
@@ -95,5 +96,5 @@
         </joint>
         <joint name="${dovetail_female_mount_prefix}body--tool0" type="fixed">
-            <origin xyz="0 0 0" rpy="0 0 0"/>
+            <origin xyz="0 0 ${dovetail_female_tool0_height}" rpy="0 0 0"/>
             <parent link="${dovetail_female_mount_prefix}body"/>
             <child link="${dovetail_female_mount_prefix}tool0"/>

File: pybullet_tree_sim/urdf/end_effectors/mock_pruner/macro/mock_pruner_macro.urdf.xacro (robot description, xacro)
@@ -5,24 +5,32 @@
     <!-- <xacro:arg name="mesh_base_path" default="./"/> -->
     <!-- <xacro:property name="end_effector_parent" value="" /> -->
+    <xacro:property name="mock_pruner_rot_offset" value="0.0 0.0 0.0"/>
     <!-- Materials -->
     <xacro:macro name="mock_pruner_macro" params="parent_link eef_prefix tof0_offset tof1_offset camera_offset mesh_base_path urdf_base_path">
         <!-- static properties -->
-        <xacro:property name="mock_pruner_mass" value="2.0" />
-        <xacro:property name="base__tool0_offset" value="0.0 0.0 0.27208"/>
+        <xacro:property name="mock_pruner_mass" value="0.256" />
+        <xacro:property name="base__tool0_offset" value="0.0 0.0050825 0.1601525"/>
         <!-- <xacro:property name="base__tool0_offset" value="0.0 0.0 0.20"/> -->
-        <xacro:property name="base__tof0_offset" value="${tof0_offset} 0 0.142"/>
-        <xacro:property name="base__tof1_offset" value="${tof1_offset} 0 0.142"/>
+        <xacro:property name="base__tof0_offset" value="${tof0_offset}"/>
+        <xacro:property name="base__tof1_offset" value="${tof1_offset}"/>
         <!-- <xacro:property name="base__tof0_offset" value="${tof0_offset} 0 0.15"/> -->
         <!-- <xacro:property name="base__tof1_offset" value="${tof1_offset} 0 0.15"/> -->
-        <xacro:property name="base__camera0_offset" value="0.0 0.0600 0.19094"/>
+        <xacro:property name="base__camera0_offset" value="-0.0017977 -0.0715747 0.0711646"/>
         <!-- additional args -->
+        <xacro:arg name="rotation_correction_plate_prefix" default="rotation_correction_plate__" />
         <xacro:arg name="dovetail_male_mount_prefix" default="dovetail_male_mount__" />
         <xacro:arg name="dovetail_female_mount_prefix" default="dovetail_female_mount__" />
         <xacro:arg name="mesh_base_path" default=""/>
-        <xacro:arg name="urdf_base_path" default=""/>
+        <!-- rotation correction plate macro -->
+        <xacro:include filename="${urdf_base_path}/end_effectors/rotation_correction_plate/macro/rotation_correction_plate_macro.urdf.xacro" />
+        <xacro:rotation_correction_plate_macro
+            parent_link="${parent_link}"
+            rotation_correction_plate_prefix="$(arg rotation_correction_plate_prefix)"
+            mesh_base_path="${mesh_base_path}"
+        />
         <!-- dovetail_mount macro -->
         <xacro:include filename="${urdf_base_path}/end_effectors/dovetail_mount/macro/dovetail_mount_macro.urdf.xacro" />
         <xacro:dovetail_mount_macro
-            parent_link="${parent_link}"
+            parent_link="$(arg rotation_correction_plate_prefix)tool0"
             dovetail_male_mount_prefix="$(arg dovetail_male_mount_prefix)"
             dovetail_female_mount_prefix="$(arg dovetail_female_mount_prefix)"
@@ -68,5 +76,5 @@
         <!-- ================== -->
         <joint name="$(arg dovetail_female_mount_prefix)tool0--${eef_prefix}base" type="fixed">
-            <origin xyz="0 0 0" rpy="0 0 0"/>
+            <origin xyz="0 0 0" rpy="${mock_pruner_rot_offset}"/>
             <parent link="$(arg dovetail_female_mount_prefix)tool0"/>
             <child link="${eef_prefix}base"/>

File: pybullet_tree_sim/urdf/end_effectors/mock_pruner/mock_pruner.urdf.xacro (robot description, xacro)
@@ -7,6 +7,6 @@
     <xacro:arg name="mock_pruner_prefix" default="mock_pruner__" />
     <xacro:arg name="mesh_base_path" default="" />
-    <xacro:arg name="tof0_offset_x" default="0.02" />
-    <xacro:arg name="tof1_offset_x" default="-0.02" />
+    <xacro:arg name="tof0_offset" default="0.1 0.0 0.142" />
+    <xacro:arg name="tof1_offset" default="-0.1 0.0 0.142" />
     <!-- mock_pruner macro -->
     <xacro:include filename="./macro/mock_pruner_macro.urdf.xacro" />
@@ -14,6 +14,6 @@
         parent_link="$(arg mock_pruner_parent_link)"
         eef_prefix="$(arg mock_pruner_prefix)"
-        tof0_offset='$(arg tof0_offset_x)'
-        tof1_offset='$(arg tof1_offset_x)'
+        tof0_offset='$(arg tof0_offset)'
+        tof1_offset='$(arg tof1_offset)'
         mesh_base_path="$(arg mesh_base_path)"
         camera_offset=''

File: pybullet_tree_sim/urdf/end_effectors/mock_pruner/test.urdf (robot description, URDF)
Before this commit: robot mock_pruner, 6 links, 4 joints
Links:
- added link dovetail_female_mount__base
- added link dovetail_female_mount__body, mass 0.025; collision mesh filename=file:///home/luke/branch_detection_ws/install/branch_detect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; visual mesh filename=file:///home/luke/branch_detection_ws/install/branch_detect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
- added link dovetail_female_mount__tool0
- added link dovetail_male_mount__base
- added link dovetail_male_mount__body, mass 0.025; collision mesh filename=file:///home/luke/branch_detection_ws/install/branch_detect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; visual mesh filename=file:///home/luke/branch_detection_ws/install/branch_detect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
- added link dovetail_male_mount__tool0
- added link rotation_correction_plate__base
- added link rotation_correction_plate__body, mass 0.003; collision mesh filename=file:///home/luke/branch_detection_ws/install/branch_detect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; visual mesh filename=file:///home/luke/branch_detection_ws/install/branch_detect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
- added link rotation_correction_plate__tool0
- link mock_pruner__base: geometry collision mesh filename=file:///home/luke/branch_detection_ws/install/branch_detect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; visual mesh filename=file:///home/luke/branch_detection_ws/install/branch_detect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
Joints:
- removed joint mock_pruner__base__camera0_joint
- removed joint mock_pruner__base__tof0_joint
- removed joint mock_pruner__base__tof1_joint
- removed joint world__mock_pruner__base
- added joint dovetail_female_mount__base--body: type fixed, parent dovetail_female_mount__base, child dovetail_female_mount__body, origin xyz=0 0 0 rpy=0 0 0
- added joint dovetail_female_mount__body--tool0: type fixed, parent dovetail_female_mount__body, child dovetail_female_mount__tool0, origin xyz=0 0 0 rpy=0 0 0
- added joint dovetail_female_mount__tool0--mock_pruner__base: type fixed, parent dovetail_female_mount__tool0, child mock_pruner__base, origin xyz=0 0 0 rpy=0 0 0
- added joint dovetail_male_mount__base--body: type fixed, parent dovetail_male_mount__base, child dovetail_male_mount__body, origin xyz=0 0 0 rpy=0 0 0
- added joint dovetail_male_mount__body--tool0: type fixed, parent dovetail_male_mount__body, child dovetail_male_mount__tool0, origin xyz=0 0 0.008 rpy=0 0 0
- added joint dovetail_male_mount__tool0--dovetail_female_mount__base: type fixed, parent dovetail_male_mount__tool0, child dovetail_female_mount__base, origin xyz=0 0 0.023 rpy=0 0 0
- added joint mock_pruner__base--camera0: type fixed, parent mock_pruner__base, child mock_pruner__camera0, origin xyz=0.0 -0.069 0.16379 rpy=0 0 0
- added joint mock_pruner__base--tof0: type fixed, parent mock_pruner__base, child mock_pruner__tof0, origin xyz=0.1 0.0 0.142 rpy=0 0 0
- added joint mock_pruner__base--tof1: type fixed, parent mock_pruner__base, child mock_pruner__tof1, origin xyz=-0.1 0.0 0.142 rpy=0 0 0
- added joint mock_pruner__base--tool0: type fixed, parent mock_pruner__base, child mock_pruner__tool0, origin xyz=0.0 0.0 0.23508 rpy=0 0 0
- added joint rotation_correction_plate__base--body: type fixed, parent rotation_correction_plate__base, child rotation_correction_plate__body, origin xyz=0 0 0 rpy=0 0 0
- added joint rotation_correction_plate__body--tool0: type fixed, parent rotation_correction_plate__body, child rotation_correction_plate__tool0, origin xyz=0 0 0.01268 rpy=0 0 0
- added joint rotation_correction_plate__tool0--dovetail_male_mount__base: type fixed, parent rotation_correction_plate__tool0, child dovetail_male_mount__base, origin xyz=0 0 0 rpy=0.0 0.0 0.0
- added joint world--mock_pruner__base: type fixed, parent world, child mock_pruner__base, origin xyz=0.0 180.0 0.0 rpy=0 0 0
- added joint world--rotation_correction_plate__base: type fixed, parent world, child rotation_correction_plate__base, origin xyz=0 0 0 rpy=0.0 0.0 0.0

File: pybullet_tree_sim/urdf/robot/generic/robot.urdf.xacro (robot description, xacro)
@@ -128,6 +128,6 @@
                 <xacro:arg name="mock_pruner_prefix" default="mock_pruner__" />
                 <xacro:arg name="mesh_base_path" default="" />
-                <xacro:arg name="tof0_offset_x" default="0.02" />
-                <xacro:arg name="tof1_offset_x" default="-0.02" />
+                <xacro:arg name="tof0_offset" default="0.1 0.0 0.142" />
+                <xacro:arg name="tof1_offset" default="-0.1 0.0 0.142"/>
                 <!-- mock_pruner  -->
                 <xacro:mock_pruner_macro
@@ -136,6 +136,6 @@
                     mesh_base_path="$(arg mesh_base_path)"
                     urdf_base_path="$(arg urdf_base_path)"
-                    tof0_offset='$(arg tof0_offset_x)'
-                    tof1_offset='$(arg tof1_offset_x)'
+                    tof0_offset='$(arg tof0_offset)'
+                    tof1_offset='$(arg tof1_offset)'
                     camera_offset=''
                 />

File: pybullet_tree_sim/urdf/shapes/cylinder/cylinder.urdf (robot description, URDF)
Before this commit: robot cylinder, 2 links, 1 joints
Links:
- link cylinder: geometry collision cylinder length=2.85 radius=0.0508; visual cylinder length=2.85 radius=0.0508

File: pybullet_tree_sim/urdf/tmp/robot.urdf (robot description, URDF)
Before this commit: robot pruning_robot, 27 links, 26 joints
Links:
- removed link cart__base
- removed link cart__cart
- removed link cart__tool0
- added link rotation_correction_plate__base
- added link rotation_correction_plate__body, mass 0.047; collision mesh filename=/home/luke/dev/pybullet/pybullet-tree-sim/pybullet_tree_sim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; visual mesh filename=/home/luke/dev/pybullet/pybullet-tree-sim/pybullet_tree_sim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
- added link rotation_correction_plate__tool0
- link dovetail_female_mount__body: mass 0.025 -> 0.038
- link dovetail_male_mount__body: mass 0.025 -> 0.033
- link mock_pruner__base: mass 2.0 -> 0.256
Joints:
- removed joint cart__base--cart__cart
- removed joint cart__cart--cart__tool0
- removed joint ur5e__tool0--dovetail_male_mount__base
- removed joint world--cart__base
- added joint rotation_correction_plate__base--body: type fixed, parent rotation_correction_plate__base, child rotation_correction_plate__body, origin xyz=0 0 0 rpy=0 0 0
- added joint rotation_correction_plate__body--tool0: type fixed, parent rotation_correction_plate__body, child rotation_correction_plate__tool0, origin xyz=0 0 0.01268 rpy=0 0 0
- added joint rotation_correction_plate__tool0--dovetail_male_mount__base: type fixed, parent rotation_correction_plate__tool0, child dovetail_male_mount__base, origin xyz=0 0 0 rpy=0.0 0.0 0.0
- added joint ur5e__tool0--rotation_correction_plate__base: type fixed, parent ur5e__tool0, child rotation_correction_plate__base, origin xyz=0 0 0 rpy=0.0 0.0 0.0
- joint dovetail_female_mount__body--tool0: origin xyz=0 0 0 rpy=0 0 0 -> xyz=0 0 0.008 rpy=0 0 0
- joint dovetail_female_mount__tool0--mock_pruner__base: origin xyz=0 0 0 rpy=0 0 0 -> xyz=0 0 0 rpy=0.0 0.0 0.0
- joint dovetail_male_mount__body--tool0: origin xyz=0 0 0.008 rpy=0 0 0 -> xyz=0 0 0.02293 rpy=0 0 0
- joint dovetail_male_mount__tool0--dovetail_female_mount__base: origin xyz=0 0 0.023 rpy=0 0 0 -> xyz=0 0 0.0 rpy=0.0 0.0 0.0
- joint mock_pruner__base--camera0: origin xyz=0.0 0.0600 0.19094 rpy=0 0 0 -> xyz=-0.0017977 -0.0715747 0.0711646 rpy=0 0 0
- joint mock_pruner__base--tof0: origin xyz=0.1 0 0.142 rpy=0 0 0 -> xyz=0.10 -0.025 0.2 rpy=0 0 0
- joint mock_pruner__base--tof1: origin xyz=-0.1 0 0.142 rpy=0 0 0 -> xyz=-0.10 -0.025 0.2 rpy=0 0 0
- joint mock_pruner__base--tool0: origin xyz=0.0 0.0 0.27208 rpy=0 0 0 -> xyz=0.0 0.0050825 0.1601525 rpy=0 0 0
- joint ur5e__base_joint: parent cart__tool0 -> amiga__tool0
