Commit message: updated Tree URDF to fix tree_id string

File: pybullet_tree_sim/urdf/trees/envy/macro/tree_macro.urdf.xacro (robot description, xacro)
@@ -10,8 +10,8 @@
         <xacro:property name="mass" value="8.0" />
         <xacro:property name="scale" value="1 1 1"/>
-        <link name="${namespace}${tree_type}_tree${tree_id}">
+        <link name="${namespace}_${tree_type}_${str(tree_id).zfill(5)}">
             <visual>
                 <geometry>
-                    <mesh filename="./meshes/trees/envy/unlabeled/obj/${namespace}${tree_type}_tree${tree_id}.obj" scale="${scale}"/>
+                    <mesh filename="./meshes/trees/envy/unlabeled/obj/${namespace}_${tree_type}_${str(tree_id).zfill(5)}.obj" scale="${scale}"/>
                 </geometry>
                 <material name="LightGrey">
@@ -21,5 +21,5 @@
             <collision concave="true">
                 <geometry>
-                    <mesh filename="./meshes/trees/envy/unlabeled/obj/${namespace}${tree_type}_tree${tree_id}.obj" scale="${scale}"/>
+                    <mesh filename="./meshes/trees/envy/unlabeled/obj/${namespace}_${tree_type}_${str(tree_id).zfill(5)}.obj" scale="${scale}"/>
                 </geometry>
             </collision>
@@ -31,7 +31,7 @@
         </link>
         <link name="world"/>
-        <joint name="${namespace}${tree_type}_tree${tree_id}_joint" type="fixed">
+        <joint name="${namespace}_${tree_type}_${str(tree_id).zfill(5)}_joint" type="fixed">
             <parent link="${parent}"/>
-            <child link="${namespace}${tree_type}_tree${tree_id}"/>
+            <child link="${namespace}_${tree_type}_${str(tree_id).zfill(5)}"/>
             <origin rpy="0.0 0.0 0.0" xyz="0.0 0.0 0.0"/>
         </joint>
