Commit message: huge updates

File: pybullet_tree_sim/urdf/tmp/robot.urdf (robot description, URDF)
Before this commit: robot pruning_robot, 30 links, 29 joints
Links:
- added link linear_slider__base
- added link linear_slider__base_link, mass 20.0; collision box size=1.35 0.3 0.10; visual mesh filename=/home/luke/dev/pybullet/pybullet-tree-sim/pybullet_tree_sim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 scale=0.001 0.001 0.001
- added link linear_slider__flange
- added link linear_slider__moving_base, mass 10.0; collision box size=0.22 0.220 0.118; visual mesh filename=/home/luke/dev/pybullet/pybullet-tree-sim/pybullet_tree_sim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 scale=0.001 0.001 0.001
- added link linear_slider__tool0
Joints:
- removed joint dovetail_female_mount__base--body
- removed joint dovetail_female_mount__body--tool0
- added joint dovetail_female_mount__base--dovetail_female_mount__body: type fixed, parent dovetail_female_mount__base, child dovetail_female_mount__body, origin xyz=0 0 0 rpy=0 0 0
- added joint dovetail_female_mount__body--dovetail_female_mount__tool0: type fixed, parent dovetail_female_mount__body, child dovetail_female_mount__tool0, origin xyz=0 0 0.008 rpy=0 0 0
- added joint linear_slider__base_joint: type fixed, parent amiga__tool0, child linear_slider__base, origin xyz=0 0 0 rpy=0 0 0
- added joint linear_slider__base_link--base_joint: type fixed, parent linear_slider__base, child linear_slider__base_link, origin xyz=0 0 0 rpy=0 0 0
- added joint linear_slider__flange--tool0_joint: type fixed, parent linear_slider__flange, child linear_slider__tool0, origin xyz=0 0 0 rpy=0 0 2.356194490192345
- added joint linear_slider__joint1: type prismatic, parent linear_slider__base_link, child linear_slider__moving_base, origin xyz=0 0 0 rpy=0 0 0, axis 1 0 0, limit lower=-0.4 upper=0.4 effort=0.05 velocity=0.08333333333333
- added joint linear_slider__moving_base--flange_joint: type fixed, parent linear_slider__moving_base, child linear_slider__flange, origin xyz=0 0 0.05 rpy=0 0 0
- joint amiga__body--amiga__tool0: origin xyz=-0.225 0.323256 1.09810607 rpy=0.0 0.0 -3.9269908169872414 -> xyz=0.125 0.323256 0.99810607 rpy=0.0 0.0 0.0
- joint ur5e__base_joint: parent amiga__tool0 -> linear_slider__tool0
