Commit message: more refactor updates

File: pybullet_tree_sim/urdf/tmp/robot.urdf (robot description, URDF)
Before this commit: robot pruning_robot, 35 links, 34 joints
Links:
- removed link dovetail_female_mount__base
- removed link dovetail_female_mount__body
- removed link dovetail_female_mount__tool0
- removed link dovetail_male_mount__base
- removed link dovetail_male_mount__body
- removed link dovetail_male_mount__tool0
- removed link mock_pruner__base
- removed link mock_pruner__camera0
- removed link mock_pruner__tof0
- removed link mock_pruner__tof1
- removed link mock_pruner__tool0
- removed link rotation_correction_plate__base
- removed link rotation_correction_plate__body
- removed link rotation_correction_plate__tool0
- added link dynamic_eef__base
- added link dynamic_eef__tof0_base, mass 0.0007; collision box size=0.0127 0.02286 0.00254; visual mesh filename=/home/luke/dev/pybullet/pybullet-tree-sim/pybullet_tree_sim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 scale=1.0
- added link dynamic_eef__tof0_sensing_unit
Joints:
- removed joint dovetail_female_mount__base--dovetail_female_mount__body
- removed joint dovetail_female_mount__body--dovetail_female_mount__tool0
- removed joint dovetail_female_mount__tool0--mock_pruner__base
- removed joint dovetail_male_mount__base--body
- removed joint dovetail_male_mount__body--tool0
- removed joint dovetail_male_mount__tool0--dovetail_female_mount__base
- removed joint mock_pruner__base--camera0
- removed joint mock_pruner__base--tof0
- removed joint mock_pruner__base--tof1
- removed joint mock_pruner__base--tool0
- removed joint rotation_correction_plate__base--body
- removed joint rotation_correction_plate__body--tool0
- removed joint rotation_correction_plate__tool0--dovetail_male_mount__base
- removed joint ur5e__tool0--rotation_correction_plate__base
- added joint dynamic_eef__base--dynamic_eef__tof0_base: type fixed, parent dynamic_eef__base, child dynamic_eef__tof0_base, origin xyz=0.0 0.0 0.0 rpy=0.0 0.0 0.0
- added joint dynamic_eef__tof0_base--dynamic_eef__tof0_sensing_unit: type fixed, parent dynamic_eef__tof0_base, child dynamic_eef__tof0_sensing_unit, origin xyz=0.0001 -0.001695 0.002776 rpy=0.0 0.0 -1.57079632679
- added joint ur5e__tool0--dynamic_eef__base: type fixed, parent ur5e__tool0, child dynamic_eef__base, origin xyz=0.0 0.0 0.0 rpy=0.0 0.0 0.0
